File: op1/op1.kicad_sch (KiCad schematic)
At the start: 0 parts

Commit message: eeerr
Other:
- note added: "OPe"
Changed lines of the file:
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@@
+		)
+	)
+	(text "OPe\n"
+		(exclude_from_sim no)
+		(at 68.58 138.43 0)
+		(effects
+			(font
+				(size 1.27 1.27)
+			)
 		)
 	)
@@
 		)
 		(instances
-			(project "fevino"
+			(project "op1"
 				(path "/8469cd9a-15fe-4677-a617-64af849f0980"
 					(page "2")
@@
 		)
 		(instances
-			(project "fevino"
+			(project "op1"
 				(path "/8469cd9a-15fe-4677-a617-64af849f0980"
 					(page "3")
@@
 		)
 		(instances
-			(project "fevino"
+			(project "op1"
 				(path "/8469cd9a-15fe-4677-a617-64af849f0980"
 					(page "7")
